Commit message: Fixed an error of SG650 URDF;

File: motoman_sg650_support/urdf/sg650_macro.xacro (robot description, xacro)
@@ -21,5 +21,5 @@
       <geometry>
         <mesh filename="package://motoman_sg650_support/meshes/sg650/visual/link_1_s.stl"/>
-        <mesh filename="package://motoman_sg650_support/meshes/sg650/visual/link_1_s-cable.stl"/>
+        <!--<mesh filename="package://motoman_sg650_support/meshes/sg650/visual/link_1_s-cable.stl"/>-->
       </geometry>
       <xacro:material_yaskawa_blue/>
@@ -30,4 +30,12 @@
       </geometry>
     </collision>
+  </link>
+  <link name="${prefix}link_1_s_cable">
+    <visual>
+      <geometry>
+        <mesh filename="package://motoman_sg650_support/meshes/sg650/visual/link_1_s-cable.stl"/>
+      </geometry>
+      <xacro:material_yaskawa_blue/>
+    </visual>
   </link>
   <link name="${prefix}link_2_l">
@@ -80,4 +88,9 @@
     <limit lower="-2.3911" upper="2.3911" effort="100" velocity="7.85"/>
   </joint>
+  <joint name="${prefix}joint_1_s_cable" type="fixed">
+    <origin xyz="0 0 0" rpy="0 0 0"/>
+    <parent link="${prefix}link_1_s"/>
+    <child link="${prefix}link_1_s_cable"/>
+  </joint>
   <joint name="${prefix}joint_2_l" type="revolute">
     <parent link="${prefix}link_1_s"/>

Commit message: Modified the SG650 link model;

File: motoman_sg650_support/urdf/sg650_macro.xacro (robot description, xacro)
@@ -53,5 +53,5 @@
   </link>
   <link name="${prefix}link_3_u">
-    <visual>
+    <!--<visual>
       <geometry>
         <mesh filename="package://motoman_sg650_support/meshes/sg650/visual/link_3_u.stl"/>
@@ -63,5 +63,5 @@
         <mesh filename="package://motoman_sg650_support/meshes/sg650/collision/link_3_u.stl"/>
       </geometry>
-    </collision>
+    </collision>-->
   </link>
   <link name="${prefix}link_4_r">
